Commit message: feat: AX 로봇 모델 및 센서 구성 추가
- AX 로봇의 URDF 및 XACRO 파일에 센서 구성 추가
- Lidar 및 카메라 센서의 매크로 정의 및 설정
- Gazebo 환경을 위한 빈 월드 파일 추가
- 로봇 메쉬 분할 스크립트 추가 및 테스트 케이스 작성
- OBJ 파일 분할 및 메쉬 속성 유지 기능 구현

File: src/ax_description/urdf/physical_properties.xacro (robot description, xacro)
@@ -359,25 +359,25 @@
   <xacro:macro name="ax_physics_arm_mount_link">
     <collision name="arm_mount_link_part_00">
-      <origin xyz="-0.115 0.125 0.298" rpy="-1.57079632679 -1.57079632679 0" />
-      <geometry>
-        <box size="0.022 0.042 0.042" />
+      <origin xyz="-0.115 0.125 0.2476553" rpy="0 0 0" />
+      <geometry>
+        <box size="0.042 0.042 0.0150192" />
       </geometry>
     </collision>
     <collision name="arm_mount_link_part_01">
-      <origin xyz="-0.115 0.125 0.548" rpy="0 0 0" />
-      <geometry>
-        <box size="0.042 0.042 0.022" />
+      <origin xyz="-0.115 0.125 0.4288823" rpy="0 0 0" />
+      <geometry>
+        <box size="0.042 0.042 0.017977" />
       </geometry>
     </collision>
     <collision name="arm_mount_link_part_02">
-      <origin xyz="-0.09 0 0.513" rpy="0 0 0" />
-      <geometry>
-        <box size="0.082 0.232 0.692" />
+      <origin xyz="-0.09 0 0.4364624" rpy="0 0 0" />
+      <geometry>
+        <box size="0.082 0.232 0.5389248" />
       </geometry>
     </collision>
     <collision name="arm_mount_link_part_03">
-      <origin xyz="-0.115 0.125 0.518" rpy="0 0 2.15984526416" />
-      <geometry>
-        <box size="0.0294620036172 0.0294620036172 0.682" />
+      <origin xyz="-0.114999984082 0.125000039364 0.43934745" rpy="2.76609068983e-08 1.84823689686e-08 2.5525454798" />
+      <geometry>
+        <box size="0.0294620014355 0.0294621067267 0.533154700931" />
       </geometry>
     </collision>
@@ -389,25 +389,25 @@
     </collision>
     <collision name="arm_mount_link_part_05">
-      <origin xyz="-0.094 -0.115 0.528" rpy="0 0 0" />
-      <geometry>
-        <box size="0.014 0.082 0.682" />
+      <origin xyz="-0.094 -0.115 0.44718815" rpy="0 0 0" />
+      <geometry>
+        <box size="0.014 0.082 0.5371775" />
       </geometry>
     </collision>
     <collision name="arm_mount_link_part_06">
-      <origin xyz="0.005 -0.138 0.528" rpy="3.14159265359 2.22044604925e-16 1.57079632679" />
-      <geometry>
-        <box size="0.036 0.212 0.682" />
+      <origin xyz="0.005 -0.138 0.44718815" rpy="0 0 0" />
+      <geometry>
+        <box size="0.212 0.036 0.5371775" />
       </geometry>
     </collision>
     <collision name="arm_mount_link_part_07">
-      <origin xyz="0.01 -0.156 0.548" rpy="0 0 0" />
-      <geometry>
-        <box size="0.202 0.002 0.602" />
+      <origin xyz="0.01000005 -0.156 0.45547455" rpy="0 0 0" />
+      <geometry>
+        <box size="0.2020001 0.002 0.4813145" />
       </geometry>
     </collision>
     <collision name="arm_mount_link_part_08">
-      <origin xyz="-0.08 -0.15606565 0.778" rpy="0 0 0" />
-      <geometry>
-        <box size="0.018 0.0078687 0.102" />
+      <origin xyz="-0.08 -0.15606565 0.6289772" rpy="0 0 0" />
+      <geometry>
+        <box size="0.018 0.0078687 0.0954924" />
       </geometry>
     </collision>
@@ -437,49 +437,49 @@
     </collision>
     <collision name="arm_mount_link_part_13">
-      <origin xyz="0.104 -0.115 0.528" rpy="0 0 0" />
-      <geometry>
-        <box size="0.014 0.082 0.682" />
+      <origin xyz="0.104000050032 -0.115000000003 0.44718815" rpy="6.27744876791e-09 6.48113536172e-08 -5.01431998919e-08" />
+      <geometry>
+        <box size="0.0140000693301 0.0820000036914 0.537177500932" />
       </geometry>
     </collision>
     <inertial>
-      <origin xyz="-0.0188531409212 -0.0105569203189 0.195896551788" rpy="0 0 0" />
+      <origin xyz="-0.0175411994985 -0.00969629540333 0.167482150183" rpy="0 0 0" />
       <mass value="3" />
-      <inertia ixx="0.16654364094" iyy="0.15865225046" izz="0.0373454531605" ixy="0.00112748162678" ixz="0.0131380058637" iyz="0.0106321190592" />
+      <inertia ixx="0.113170823963" iyy="0.105283122913" izz="0.0371800064437" ixy="0.000991321541212" ixz="0.0100896144115" iyz="0.00821486435918" />
     </inertial>
   </xacro:macro>
   <xacro:macro name="ax_physics_column_link">
     <collision name="column_link_part_00">
-      <origin xyz="-5.66215664767e-09 -7.3979504122e-09 0.127" rpy="0.132133684518 -1.57079632679 0" />
-      <geometry>
-        <box size="0.016 0.209935326354 0.209935326354" />
+      <origin xyz="-2.32456185978e-10 -4.70424033467e-10 0.077689950156" rpy="-3.13689934831 -1.57079626484 0" />
+      <geometry>
+        <box size="0.011088712574 0.209997710294 0.20999771019" />
       </geometry>
     </collision>
     <collision name="column_link_part_01">
-      <origin xyz="-5.66215664785e-09 -7.39795041182e-09 0.347" rpy="0.132133684518 -1.57079632679 0" />
-      <geometry>
-        <box size="0.016 0.209935326354 0.209935326354" />
+      <origin xyz="1.84150670045e-09 3.38590378081e-09 0.234827099856" rpy="-0.0344805870107 -1.57079631089 0" />
+      <geometry>
+        <box size="0.0129108030207 0.209876358767 0.209876362169" />
       </geometry>
     </collision>
     <collision name="column_link_part_02">
-      <origin xyz="-5.66215664731e-09 -7.39795041256e-09 0.567" rpy="0.132133684518 -1.57079632679 0" />
-      <geometry>
-        <box size="0.016 0.209935326354 0.209935326354" />
+      <origin xyz="3.43734796898e-10 6.75967892343e-10 0.42059745" rpy="3.03871075006 -1.57079607625 -3.04549364055" />
+      <geometry>
+        <box size="0.0147329520166 0.209995214199 0.209995217723" />
       </geometry>
     </collision>
     <collision name="column_link_part_03">
-      <origin xyz="2.04851494747e-08 -4.39483400723e-08 0.36" rpy="0 0 1.36856145758" />
-      <geometry>
-        <box size="0.201796127569 0.201796107483 0.722" />
+      <origin xyz="4.11545618912e-08 7.88637269009e-10 0.283329299995" rpy="-3.08446987951e-08 -5.89366822012e-09 -1.65971871811" />
+      <geometry>
+        <box size="0.201535756408 0.201535662062 0.56865860626" />
       </geometry>
     </collision>
     <inertial>
-      <origin xyz="0 0 0.236" rpy="0 0 0" />
+      <origin xyz="0 0 0.18999758" rpy="0 0 0" />
       <mass value="4" />
-      <inertia ixx="0.211244333333" iyy="0.211244333333" izz="0.02795" ixy="0" ixz="0" iyz="0" />
+      <inertia ixx="0.131793586873" iyy="0.131793586873" izz="0.02795" ixy="0" ixz="0" iyz="0" />
     </inertial>
   </xacro:macro>
   <xacro:macro name="ax_physics_arm_rotating_base_link">
     <collision name="arm_rotating_base_link_part_00">
-      <origin xyz="-1.37426437143e-09 -2.96173872102e-09 -0.01" rpy="0.0292075754294 -1.57079632582 0" />
+      <origin xyz="-1.37426440617e-09 -2.96173876073e-09 -0.01" rpy="0.0292075754545 -1.57079632582 0" />
       <geometry>
         <box size="0.0220000002059 0.217907879496 0.217907876575" />
@@ -487,50 +487,62 @@
     </collision>
     <collision name="arm_rotating_base_link_part_01">
-      <origin xyz="-3.87034975921e-08 -2.09096665105e-08 0.003" rpy="2.06612516714 -1.57079632679 0" />
-      <geometry>
-        <box size="0.01 0.211997891884 0.211997803902" />
+      <origin xyz="-3.870349759e-08 -2.09096665263e-08 0.003" rpy="2.06612516751 -1.57079632679 0" />
+      <geometry>
+        <box size="0.01 0.211997891883 0.211997803902" />
       </geometry>
     </collision>
     <collision name="arm_rotating_base_link_part_02">
-      <origin xyz="-0.0689374999706 1.20668312582e-11 0.099999999306" rpy="1.58526535076 1.30581392366e-08 -7.11086189931e-10" />
-      <geometry>
-        <box size="0.0241250019783 0.157983672455 0.157983670794" />
+      <origin xyz="-0.0741566999754 2.67406740197e-12 0.100000000175" rpy="1.56788318927 1.09542175331e-08 -8.48564996048e-10" />
+      <geometry>
+        <box size="0.0280706016596 0.157999338 0.157999338081" />
       </geometry>
     </collision>
     <collision name="arm_rotating_base_link_part_03">
-      <origin xyz="-0.005 0 0.095" rpy="0 0 0" />
-      <geometry>
-        <box size="0.132 0.188 0.192" />
+      <origin xyz="0.0011828 0 0.095" rpy="0 0 0" />
+      <geometry>
+        <box size="0.155183 0.188 0.192" />
+      </geometry>
+    </collision>
+    <collision name="arm_rotating_base_link_part_04">
+      <origin xyz="0.0806530499501 4.24353531914e-13 0.100000000196" rpy="-1.57370946118 -2.21739655526e-08 4.4408920985e-16" />
+      <geometry>
+        <box size="0.0475559033594 0.157999338684 0.157999338068" />
+      </geometry>
+    </collision>
+    <collision name="arm_rotating_base_link_part_05">
+      <origin xyz="0.115894699949 -7.98881691529e-09 0.0999999549105" rpy="-1.65443926245 -2.36757160543e-08 -5.91891957669e-09" />
+      <geometry>
+        <box size="0.0446664034545 0.147711091747 0.147711190812" />
       </geometry>
     </collision>
     <inertial>
-      <origin xyz="-0.00380900779249 -7.27845350845e-10 0.0893699309651" rpy="0 0 0" />
+      <origin xyz="0.0392273753996 -8.14400927077e-10 0.0925080391138" rpy="0 0 0" />
       <mass value="1" />
-      <inertia ixx="0.00430431015514" iyy="0.00352368707856" izz="0.00294752968072" ixy="-3.1124180314e-11" ixz="3.35452101992e-05" iyz="-6.5227810357e-11" />
+      <inertia ixx="0.00394188955562" iyy="0.00429610056541" izz="0.00387231842705" ixy="-1.9468647556e-11" ixz="-0.000292559158488" iyz="-3.6238804937e-11" />
     </inertial>
   </xacro:macro>
   <xacro:macro name="ax_physics_upper_arm_link">
     <collision name="upper_arm_link_part_00">
-      <origin xyz="-0.011 3.10807474202e-08 0.559999975751" rpy="-2.23334730794 3.63947936233e-08 3.53030711331e-08" />
-      <geometry>
-        <box size="0.0120000070977 0.151954377486 0.151954421669" />
+      <origin xyz="-0.011 8.789787731e-09 0.559999951596" rpy="0.179635306985 -7.1054273576e-15 -1.09176347129e-09" />
+      <geometry>
+        <box size="0.0120000001528 0.151979065115 0.151978966724" />
       </geometry>
     </collision>
     <collision name="upper_arm_link_part_01">
-      <origin xyz="-0.0035 4.70035108058e-09 0.560000014592" rpy="-1.88242118685 -2.28734808871e-11 -4.34601243882e-10" />
-      <geometry>
-        <box size="0.0190000000655 0.157999436911 0.157999467575" />
+      <origin xyz="-0.00349999999999 1.54566109911e-10 0.560000002776" rpy="-1.62642554801 9.81448140536e-08 9.84652737124e-08" />
+      <geometry>
+        <box size="0.0190000209371 0.157758678155 0.157758683846" />
       </geometry>
     </collision>
     <collision name="upper_arm_link_part_02">
-      <origin xyz="0.002 0 0" rpy="0.944615899235 0 0" />
-      <geometry>
-        <box size="0.009 0.168884848445 0.168884848445" />
+      <origin xyz="0.002 -4.23995245766e-18 -5.00000000063e-08" rpy="0.937036052313 6.88338275268e-15 -2.17048601314e-14" />
+      <geometry>
+        <box size="0.009 0.168833143408 0.168833122046" />
       </geometry>
     </collision>
     <collision name="upper_arm_link_part_03">
-      <origin xyz="0.07 5.21000896909e-11 0.560000001613" rpy="1.57079283023 -1.53851066817 1.57079990055" />
-      <geometry>
-        <box size="0.169912460934 0.169912458918 0.142000021903" />
+      <origin xyz="0.07 -4.08547679117e-09 0.559999945101" rpy="-1.57079532592 -1.48045707802 -1.57079724458" />
+      <geometry>
+        <box size="0.16962605874 0.169625968698 0.142000019035" />
       </geometry>
     </collision>
@@ -542,7 +554,7 @@
     </collision>
     <collision name="upper_arm_link_part_05">
-      <origin xyz="0.126 1.75192876503e-10 2.95447986705e-09" rpy="-1.63002433986 -5.95381521862e-11 4.56458870701e-10" />
-      <geometry>
-        <box size="0.0140000000624 0.141754508829 0.141754514751" />
+      <origin xyz="0.126 1.5352595541e-09 -5.86258887082e-08" rpy="-1.39465799736 6.35073993394e-10 4.56458870701e-10" />
+      <geometry>
+        <box size="0.014000000106 0.141974520888 0.141974619338" />
       </geometry>
     </collision>
@@ -560,87 +572,87 @@
     </collision>
     <inertial>
-      <origin xyz="0.0530949387907 3.86465791784e-06 0.198025261645" rpy="0 0 0" />
+      <origin xyz="0.0530959773365 3.86641157046e-06 0.197929511228" rpy="0 0 0" />
       <mass value="4" />
-      <inertia ixx="0.243511691489" iyy="0.238077401263" izz="0.0141682587197" ixy="-1.04125897713e-06" ixz="-0.00630743376914" iyz="4.36105180371e-07" />
+      <inertia ixx="0.243404953883" iyy="0.23797260736" izz="0.0141651928423" ixy="-1.04190681572e-06" ixz="-0.00630144583047" iyz="4.3588000646e-07" />
     </inertial>
   </xacro:macro>
   <xacro:macro name="ax_physics_forearm_link">
     <collision name="forearm_link_part_00">
-      <origin xyz="0.084 0.455000100413 -0.440000062036" rpy="-1.57081035548 1.55991604412 -1.57081023583" />
-      <geometry>
-        <box size="0.133992286955 0.133992206117 0.170000023779" />
+      <origin xyz="0.084 0.455000097541 -0.440000115025" rpy="1.57080271107 1.54186776052 1.57080282723" />
+      <geometry>
+        <box size="0.13394497088 0.133944788999 0.170000026966" />
       </geometry>
     </collision>
     <collision name="forearm_link_part_01">
-      <origin xyz="0.0500000510432 0.219592676503 -0.212353324298" rpy="-2.33943620449 6.80809457698e-08 6.80299760969e-08" />
-      <geometry>
-        <box size="0.102000039468 0.177999969559 0.788949377305" />
+      <origin xyz="0.0500000803606 0.219592679052 -0.212353321662" rpy="-2.33943619248 6.48790865476e-09 7.88374410199e-08" />
+      <geometry>
+        <box size="0.102000008793 0.177999828697 0.788949375202" />
       </geometry>
     </collision>
     <collision name="forearm_link_part_02">
-      <origin xyz="0.114 9.99999999924e-08 -1.37959498667e-18" rpy="-1.54756137939 3.65787333756e-09 -1.54657292528e-08" />
-      <geometry>
-        <box size="0.0300000026117 0.173953578605 0.173953574213" />
+      <origin xyz="0.114 9.34087947333e-08 -4.36343829041e-10" rpy="-1.50469186695 4.00596822381e-09 -3.69916419718e-09" />
+      <geometry>
+        <box size="0.0300000008979 0.173624347351 0.173624347356" />
       </geometry>
     </collision>
     <collision name="forearm_link_part_03">
-      <origin xyz="0.101 0.15925 -0.154" rpy="-0.802156066702 0 3.14159265359" />
-      <geometry>
-        <box size="0.002 0.0919999899066 0.182000049329" />
+      <origin xyz="0.101 0.15925 -0.15400005" rpy="-0.802155809235 0 3.14159265359" />
+      <geometry>
+        <box size="0.002 0.0920001081362 0.182000142017" />
       </geometry>
     </collision>
     <collision name="forearm_link_part_04">
-      <origin xyz="0.128535900003 2.16927220621e-08 -3.31674473357e-08" rpy="0.400652778725 -1.30826061095e-09 4.00666333444e-10" />
-      <geometry>
-        <box size="0.016928200197 0.165994832446 0.165994740365" />
+      <origin xyz="0.128535900317 5.28533045592e-08 -1.02571666031e-07" rpy="-2.30304483816 1.12514680684e-07 1.11424703242e-07" />
+      <geometry>
+        <box size="0.0169282228023 0.16583370855 0.16583370855" />
       </geometry>
     </collision>
     <collision name="forearm_link_part_05">
-      <origin xyz="0.1355 4.99999999991e-08 1.81767976525e-19" rpy="0.77470382597 0 0" />
-      <geometry>
-        <box size="0.005 0.0199990094429 0.0199990109553" />
+      <origin xyz="0.1355 9.99999999996e-08 -9.99999999989e-08" rpy="-0.180443166657 0 0" />
+      <geometry>
+        <box size="0.005 0.0199950935842 0.0199950935842" />
       </geometry>
     </collision>
     <collision name="forearm_link_part_06">
-      <origin xyz="0.168401950009 0.455000038511 -0.440000071035" rpy="1.07091085504 3.95094756911e-09 -4.20688306413e-09" />
-      <geometry>
-        <box size="0.0131961006057 0.121995078047 0.12199512598" />
+      <origin xyz="0.16840195001 0.45500001057 -0.440000107279" rpy="0.967917604835 4.93316765215e-09 -4.20688361924e-09" />
+      <geometry>
+        <box size="0.0131961006806 0.121988381609 0.121988520682" />
+      </geometry>
+    </collision>
+    <collision name="forearm_link_part_07">
+      <origin xyz="0.171 0.455000105214 -0.440000115281" rpy="-1.24197071942 -1.60428692553e-09 -2.99482771915e-10" />
+      <geometry>
+        <box size="0.0080000001341 0.085991039117 0.0859910068181" />
       </geometry>
     </collision>
     <inertial>
-      <origin xyz="0.0786578564106 0.158503844461 -0.15327842046" rpy="0 0 0" />
+      <origin xyz="0.0788686011554 0.158950793081 -0.153710639244" rpy="0 0 0" />
       <mass value="3" />
-      <inertia ixx="0.21017374323" iyy="0.106569182582" izz="0.113196395981" ixy="0.00766186902224" ixz="-0.00740927882079" iyz="0.0988278635101" />
+      <inertia ixx="0.210713841069" iyy="0.106869979478" izz="0.113516101115" ixy="0.00748717009587" ixz="-0.00724033844235" iyz="0.099109959977" />
     </inertial>
   </xacro:macro>
   <xacro:macro name="ax_physics_wrist_link">
     <collision name="wrist_link_part_00">
-      <origin xyz="2.61345425518e-08 -4.23033232569e-08 -0.217000007483" rpy="-0.894715817063 1.57079505632 2.14064466274" />
-      <geometry>
-        <box size="0.11600015803 0.141819116797 0.141819112798" />
+      <origin xyz="-1.6706919313e-07 -4.61676704378e-08 -0.217000007785" rpy="-0.907452739814 1.57079500738 2.19615027353" />
+      <geometry>
+        <box size="0.116000164398 0.141899012262 0.141899007627" />
       </geometry>
     </collision>
     <collision name="wrist_link_part_01">
-      <origin xyz="8.47607090067e-06 -5.40440883682e-06 -0.196" rpy="1.51317674725 -1.57079632093 0" />
-      <geometry>
-        <box size="0.0540000007501 0.137975702855 0.137988950269" />
+      <origin xyz="0.0004998 0 -0.0875" rpy="0 0 0" />
+      <geometry>
+        <box size="0.137 0.132 0.147" />
       </geometry>
     </collision>
     <collision name="wrist_link_part_02">
-      <origin xyz="0.0005 0 -0.0875" rpy="0 0 0" />
-      <geometry>
-        <box size="0.137 0.132 0.147" />
-      </geometry>
-    </collision>
-    <collision name="wrist_link_part_03">
-      <origin xyz="3.24811685251e-18 1.20079592939e-18 -0.248" rpy="2.06046003607 -1.5707963264 0" />
-      <geometry>
-        <box size="0.0100000000463 0.125999878926 0.125999878926" />
+      <origin xyz="-1.99999999996e-07 5.11328643967e-18 -0.248" rpy="2.02115128794 -1.5707963261 0" />
+      <geometry>
+        <box size="0.0100000000805 0.125898192438 0.125898192438" />
       </geometry>
     </collision>
     <inertial>
-      <origin xyz="0.000119106074289 -5.03419164693e-07 -0.127719976378" rpy="0 0 0" />
+      <origin xyz="0.000141778496886 -1.1510535167e-08 -0.123627502181" rpy="0 0 0" />
       <mass value="1" />
-      <inertia ixx="0.00536804009663" iyy="0.00539458185429" izz="0.00230032963235" ixy="-1.66088591694e-09" ixz="-4.70549050194e-06" iyz="-3.46812243073e-08" />
+      <inertia ixx="0.00547928019442" iyy="0.00551113578034" izz="0.0022997830219" ixy="-2.67110170803e-12" ixz="-5.12793302094e-06" iyz="-1.22321637319e-09" />
     </inertial>
   </xacro:macro>
