Commit message: feat: AX_1 및 AX_2의 센서 및 카메라 구성 변경
- AX_1의 arm_rgbd 및 arm_rgb 카메라의 부모 링크를 각각 wrist_link와 upper_arm_link로 설정
- suction 공구에 대해 arm_rgbd 카메라의 위치 및 방향을 조정
- suction_tof 센서를 suction_base_link에 추가하여 흡착 공구에서만 사용 가능하도록 설정
- sensor_mounts.yaml 파일에 새로운 센서 배치 및 속성 추가
- 관련 테스트 케이스를 추가하여 새로운 센서 구성 검증

File: src/ax_description/urdf/ax.urdf.xacro (robot description, xacro)
@@ -477,5 +477,7 @@
         </xacro:ax_suction_gripper>
     </xacro:if>
-    <xacro:ax_sensor_suite profile="ax1" robot_id="$(arg sensor_robot_id)" frame_prefix="${frames}"/>
+    <!-- tool selects the arm_rgbd mount (plate centre for suction, wrist otherwise). -->
+    <xacro:ax_sensor_suite profile="ax1" robot_id="$(arg sensor_robot_id)" frame_prefix="${frames}"
+                           tool="$(arg gripper_model)"/>
     <!-- 4개 바퀴를 좌우 쌍으로 구동하는 차동 구동 시스템: 바퀴 간격과 반지름으로 주행 계산 -->
     <!-- 모델 ax의 기본 명령 토픽은 /model/${model_name}/cmd_vel. ROS /cmd_vel과의 연결은 launch 브리지가 담당한다. -->

File: src/ax_description/urdf/sensors.xacro (robot description, xacro)
@@ -35,4 +35,5 @@
     </joint>
   </xacro:macro>
+  <!-- 2D LiDAR: 링크 +X 기준 ±90°(전방 180°)를 수평면에서 스캔한다. -->
   <xacro:macro name="ax_lidar" params="name xyz rpy topic_prefix frame_prefix">
     <xacro:ax_sensor_body
@@ -64,4 +65,45 @@
             <max>10</max>
             <resolution>0.01</resolution>
+          </range>
+        </lidar>
+      </sensor>
+    </gazebo>
+  </xacro:macro>
+  <!-- 근거리 ToF 근사: 링크 +X 한 방향의 단일 광선(gpu_lidar 1샘플)이다. 특정 실물 ToF의
+       정확도·재질 응답·다중 경로 오차를 재현하지 않는다. 범위 밖·무효 값은 Gazebo가 inf로
+       내보내며 0이나 접촉 성공으로 바꾸지 않는다. ROS에는 원시 inf를 보존하는 1빔
+       sensor_msgs/msg/LaserScan(ranges[0], 단위 m, 센서 원점 기준)으로 전달한다. 설치된
+       ros_gz_bridge의 LaserScan->Range 변환은 +inf를 max_range + 1(현재 1.5 m)이라는 범위 밖
+       유한값으로 바꾸므로 쓰지 않는다. -->
+  <xacro:macro name="ax_tof" params="name parent xyz rpy min_range max_range topic_prefix frame_prefix">
+    <!-- 0.012 m(측정 방향) x 0.02 x 0.02 m, 0.01 kg 개발용 외형 -->
+    <xacro:ax_sensor_body
+        name="${name}"
+        parent="${parent}"
+        xyz="${xyz}"
+        rpy="${rpy}"
+        mass="0.01"
+        sx="0.012"
+        sy="0.02"
+        sz="0.02"/>
+    <gazebo reference="${name}_link">
+      <sensor name="${name}" type="gpu_lidar">
+        <topic>${topic_prefix}/${name}/scan</topic>
+        <gz_frame_id>${frame_prefix}${name}_link</gz_frame_id>
+        <always_on>true</always_on>
+        <update_rate>30</update_rate>
+        <lidar>
+          <scan>
+            <horizontal>
+              <samples>1</samples>
+              <resolution>1</resolution>
+              <min_angle>0</min_angle>
+              <max_angle>0</max_angle>
+            </horizontal>
+          </scan>
+          <range>
+            <min>${min_range}</min>
+            <max>${max_range}</max>
+            <resolution>0.001</resolution>
           </range>
         </lidar>
@@ -116,7 +158,11 @@
     </gazebo>
   </xacro:macro>
-  <xacro:macro name="ax_sensor_suite" params="profile robot_id frame_prefix">
+  <!-- tool: gripper_model of the AX_1 arm. Only the suction tool has suction_base_link,
+       so the plate-centre RGB-D mount is used there and the wrist mount otherwise. -->
+  <xacro:macro name="ax_sensor_suite" params="profile robot_id frame_prefix tool:=none">
     <xacro:property name="mounts" value="${xacro.load_yaml('../config/sensor_mounts.yaml')[profile]}"/>
     <xacro:property name="topics" value="${'/ax/' + robot_id + '/sensors'}"/>
+    <!-- 몸체 전방: 카메라(front_rgb, +Y)–LiDAR(중앙)–카메라(front_rgbd, -Y)를
+         같은 높이에 둔다. 좌표는 base_link 기준 m, 모두 로봇 +X를 향한다. -->
     <xacro:ax_lidar
         name="front_lidar"
@@ -166,15 +212,37 @@
     </gazebo>
     <xacro:if value="${profile == 'ax1'}">
+      <!-- 팔 카메라의 부모 링크와 좌표는 sensor_mounts.yaml에서 함께 읽는다.
+           xyz/rpy는 해당 부모 링크 좌표계 기준이므로 부모만 바꿔 재사용하지 않는다. -->
+      <!-- arm_rgbd: 모든 공구에서 wrist_link 바깥쪽(+Y)에 둔다. suction은 흡착판 바깥의
+           상자 윗면을 비스듬히 보는 별도 좌표, 다른 공구는 기존 손목 좌표를 쓴다.
+           접근 전 물체 표면·높이·주변 형상 관찰용이며 최종 접근 거리는 suction_tof가 맡는다. -->
+      <xacro:property name="rgbd_mount"
+                      value="${mounts['arm_rgbd'] if tool == 'suction' else mounts['arm_rgbd_non_suction']}"/>
       <xacro:ax_camera
           name="arm_rgbd"
-          parent="wrist_link"
+          parent="${rgbd_mount['parent']}"
           depth="${True}"
-          xyz="${mounts['arm_rgbd']['xyz']}"
-          rpy="${mounts['arm_rgbd']['rpy']}"
+          xyz="${rgbd_mount['xyz']}"
+          rpy="${rgbd_mount['rpy']}"
           topic_prefix="${topics}"
           frame_prefix="${frame_prefix}"/>
+      <!-- suction_tof: 흡착 공구에서만 4컵 중앙에 생성하고 말단 회전과 함께 돈다.
+           최종 접근 간격 = 측정 거리 - lip_offset(센서 원점에서 컵 끝면까지). -->
+      <xacro:if value="${tool == 'suction'}">
+        <xacro:ax_tof
+            name="suction_tof"
+            parent="${mounts['suction_tof']['parent']}"
+            xyz="${mounts['suction_tof']['xyz']}"
+            rpy="${mounts['suction_tof']['rpy']}"
+            min_range="${mounts['suction_tof']['min_range']}"
+            max_range="${mounts['suction_tof']['max_range']}"
+            topic_prefix="${topics}"
+            frame_prefix="${frame_prefix}"/>
+      </xacro:if>
+      <!-- arm_rgb: upper_arm_link. 공구 말단·물체 접촉 장면을 관찰하는 영상이며
+           흡착·접촉 성공 판정 센서가 아니다. -->
       <xacro:ax_camera
           name="arm_rgb"
-          parent="wrist_link"
+          parent="${mounts['arm_rgb']['parent']}"
           depth="${False}"
           xyz="${mounts['arm_rgb']['xyz']}"

Commit message: feat: AX 로봇 모델의 .gitignore 및 문서 업데이트
- .gitignore에 로컬 Archify 소스 및 관련 파일 추가
- README.md에 AX 전체 시스템 구성도 이미지 추가
- AX_5DOF_ARM_SPEC.md에서 effort 값 및 설명 업데이트
- INTERFACES.md에서 어깨 처짐 현상에 대한 설명 수정
- ax.urdf.xacro에서 각 관절의 effort 값을 개발용 잠정값으로 수정

File: src/ax_description/urdf/ax.urdf.xacro (robot description, xacro)
@@ -296,6 +296,6 @@
         <!-- 원형 축 형상에서 추정한 X축 회전. 확정 기구 사양은 별도 확인한다. -->
         <axis xyz="1 0 0"/>
-        <!-- AX v0.1 속도 제한 적용. 위치 범위 유지, effort는 토크 산정 전의 미검증 기존값. -->
-        <limit lower="-1.5708" upper="1.5708" effort="20.0" velocity=".50"/>
+        <!-- AX v0.1 속도 제한 적용. 위치 범위 유지. effort는 정적 토크 계산(팔 사양 6.1절)으로 정한 개발용 잠정값이며 실물 모터 정격이 아니다. -->
+        <limit lower="-1.5708" upper="1.5708" effort="100" velocity=".50"/>
         <dynamics damping="2.0" friction="0.0"/>
     </joint>
@@ -320,6 +320,6 @@
         <origin xyz="0.132 0 0.56" rpy="0 0 0"/>
         <axis xyz="1 0 0"/>
-        <!-- AX v0.1 속도 제한 적용. 위치 범위 유지, effort는 토크 산정 전의 미검증 기존값. -->
-        <limit lower="-2.0" upper="2.0" effort="15" velocity=".50"/>
+        <!-- AX v0.1 속도 제한 적용. 위치 범위 유지. effort는 정적 토크 계산(팔 사양 6.1절)으로 정한 개발용 잠정값이며 실물 모터 정격이 아니다. -->
+        <limit lower="-2.0" upper="2.0" effort="65" velocity=".50"/>
         <dynamics damping="1.0" friction="0.0"/>
     </joint>
@@ -344,6 +344,6 @@
         <origin xyz="0.09 0.455 -0.44" rpy="0 0 0"/>
         <axis xyz="1 0 0"/>
-        <!-- AX v0.1 속도 제한 적용. 위치 범위 유지, effort는 토크 산정 전의 미검증 기존값. -->
-        <limit lower="-1.57" upper="1.57" effort="5" velocity=".70"/>
+        <!-- AX v0.1 속도 제한 적용. 위치 범위 유지. effort는 정적 토크 계산(팔 사양 6.1절)으로 정한 개발용 잠정값이며 실물 모터 정격이 아니다. -->
+        <limit lower="-1.57" upper="1.57" effort="25" velocity=".70"/>
         <dynamics damping="0.3" friction="0.0"/>
     </joint>
@@ -496,5 +496,5 @@
         <xacro:ax_velocity_joint name="rear_left_wheel_joint"/>
         <xacro:ax_velocity_joint name="rear_right_wheel_joint"/>
-        <!-- 팔 위치 범위·속도·effort 상한은 각 joint의 limit을 따른다(effort는 토크 산정 전 미검증 값). -->
+        <!-- 팔 위치 범위·속도·effort 상한은 각 joint의 limit을 따른다(어깨·팔꿈치·손목 effort는 개발용 잠정값, 기둥 yaw·말단 회전은 미검증 기존값). -->
         <xacro:ax_position_joint name="column_yaw_joint"/>
         <xacro:ax_position_joint name="shoulder_joint"/>
